Commit message: 重建为省赛 4.2m×4.2m 场地（替换总决赛全城场景）
- 场地：4.2m 方形地板 + 四周围墙（厚0.5cm、高50cm）
- 环形闭合车道（边线+中心虚线，留白60cm、路宽40cm）+ 橙黄方向箭头
- 2组红绿灯（48×64cm 箱体带双腿）+ 停止线 + 下方灯北侧斑马线；黄灯改5s
- 18人偶立牌（15×5cm）：A街区6 + B街区6 + 人行道6（含F1/F2非社区）
- 右侧3车位（3/2/1号）+ 车背景立牌(34.5×25cm)+车牌(9.5×3cm)，额外1车背景
- 机器人缩至适合40cm车道；lidar 6m、相机100°FOV
- 素材来自 D:\\DESK\\复赛资料，generate_textures/world 全部重写

File: src/smart_community_sim/robot/robot.xacro (robot description, xacro)
@@ -6,12 +6,12 @@
 -->
 <robot name="robot" xmlns:xacro="http://www.ros.org/wiki/xacro">
-  <!-- ===== 尺寸/质量参数 ===== -->
-  <xacro:property name="wheel_radius" value="0.05"/>
-  <xacro:property name="wheel_width" value="0.03"/>
-  <xacro:property name="wheel_separation" value="0.30"/>  <!-- 左右轮横向间距 -->
-  <xacro:property name="base_length" value="0.30"/>
-  <xacro:property name="base_width" value="0.20"/>
-  <xacro:property name="base_height" value="0.10"/>
-  <xacro:property name="caster_radius" value="0.025"/>
+  <!-- ===== 尺寸/质量参数（省赛 4.2m 场地，缩小底盘以便通过 40cm 车道） ===== -->
+  <xacro:property name="wheel_radius" value="0.03"/>
+  <xacro:property name="wheel_width" value="0.02"/>
+  <xacro:property name="wheel_separation" value="0.18"/>  <!-- 左右轮横向间距 -->
+  <xacro:property name="base_length" value="0.20"/>
+  <xacro:property name="base_width" value="0.14"/>
+  <xacro:property name="base_height" value="0.08"/>
+  <xacro:property name="caster_radius" value="0.02"/>
   <xacro:property name="chassis_mass" value="3.0"/>
   <xacro:property name="wheel_mass" value="0.2"/>
@@ -174,5 +174,5 @@
         <range>
           <min>0.1</min>
-          <max>12</max>
+          <max>6</max>
           <resolution>0.01</resolution>
         </range>
@@ -186,5 +186,5 @@
       <update_rate>30</update_rate>
       <camera>
-        <horizontal_fov>1.0471975</horizontal_fov>
+        <horizontal_fov>1.745329</horizontal_fov>
         <image>
           <width>640</width>
@@ -193,5 +193,5 @@
         <clip>
           <near>0.05</near>
-          <far>100</far>
+          <far>10</far>
         </clip>
       </camera>

Commit message: 合并导航组代码 + 修复仿真/导航问题
- 仿真：底盘抬高0.02、DiffDrive显式cmd_vel话题、GPU后端自动检测/dev/dxg、移除6块路面薄板碰撞体
- 导航：ROS_DISTRO humble→jazzy、移除opennav_docking的docking_server、巡检target字段透传、去~/ros2_ws硬编码
- 新增视觉组接口文档 docs/vision_interface.md

File: src/smart_community_sim/robot/robot.xacro (robot description, xacro)
@@ -29,8 +29,11 @@
   <link name="base_link">
     <visual>
+      <!-- 底盘盒抬高 0.02，避免底部低于轮底导致车趴地、轮子悬空空转 -->
+      <origin xyz="0 0 0.02"/>
       <geometry><box size="${base_length} ${base_width} ${base_height}"/></geometry>
       <material name="chassis_blue"/>
     </visual>
     <collision>
+      <origin xyz="0 0 0.02"/>
       <geometry><box size="${base_length} ${base_width} ${base_height}"/></geometry>
     </collision>
@@ -136,4 +139,7 @@
       <wheel_separation>${wheel_separation}</wheel_separation>
       <wheel_radius>${wheel_radius}</wheel_radius>
+      <!-- 显式指定速度指令话题：部分 gz-sim 版本/机器上默认话题名不是
+           /model/robot/cmd_vel，会导致 bridge 发进来的 cmd_vel 车不动 -->
+      <topic>/model/robot/cmd_vel</topic>
       <odom_publish_frequency>50</odom_publish_frequency>
       <odom_topic>/model/robot/diffdrive_odom</odom_topic>
